Commit message: Goal 4 Complete

File: vision_rpi_bot/urdf/vision_rpi_bot_lf.urdf (robot description, URDF)
Before this commit: robot vision_rpi_bot, 9 links, 8 joints
Links:
- removed link lidar_link
Joints:
- removed joint lidar_joint
- joint camera_joint: origin xyz=0 -0.18 0.2 rpy=0.0 0 -1.57 -> xyz=0 -0.24 0.2 rpy=0.0 0.65 -1.57
